Commit message: moveit configured

File: iri_table_clearing_description/xacro/grippertcp.urdf.xacro (robot description, xacro)
@@ -10,4 +10,6 @@
   <xacro:property name="finger_deep" value="0.025" />
   <xacro:property name="closing_width" value="0.025" />
+  <!-- This offset is due to avoid the collision between the gripper and the end effector "boundary"-->
+  <xacro:property name="offset" value="0.0051" />
   <xacro:macro name="grippertcp" params="prefix parent">
     <link name="${prefix}_link_gripper_tcp" />
@@ -20,5 +22,5 @@
       <parent link="${parent}" />
       <child link="${prefix}_link_gripper_base_tcp" />
-      <origin xyz="0.0 0.0 ${height/2}" rpy="0 0 0" />
+      <origin xyz="0.0 0.0 ${height/2 + offset/2}" rpy="0 0 0" />
     </joint>
     <joint name="${prefix}_joint_gripper_left_finger_tcp" type="fixed" >
@@ -36,5 +38,5 @@
 	      <origin xyz="0 0 0" rpy="0 0 0"/>
 	      <geometry>
-		<box size="${width} ${deep} ${height}"/>
+		<box size="${width} ${deep} ${height -offset}"/>
 	      </geometry>
 	    </collision>
@@ -42,5 +44,5 @@
 	      <origin xyz="0 0 0" rpy="0 0 0"/>
 	      <geometry>
-		<box size="${width} ${deep} ${height}"/>
+		<box size="${width} ${deep} ${height -offset}"/>
 	      </geometry>
 	      <material name="white"/>

Commit message: - Added grasping service, TODO: add the service to open and close the gripper and to send the robot to the bin - IK unfeasible grasp predicate done.

File: iri_table_clearing_description/xacro/grippertcp.urdf.xacro (robot description, xacro)
@@ -3,11 +3,11 @@
   <xacro:property name="M_PI" value="3.1415926535897931" />
   <xacro:property name="mass" value="0.05" /> <!-- arbitrary value for mass -->
-  <xacro:property name="height" value="0.07" />
-  <xacro:property name="width" value="0.065" />
-  <xacro:property name="deep" value="0.06" />
-  <xacro:property name="finger_height" value="0.045" />
-  <xacro:property name="finger_width" value="0.02" />
-  <xacro:property name="finger_deep" value="0.025" />
-  <xacro:property name="closing_width" value="0.025" />
+  <xacro:property name="height" value="0.07" /> <!-- z axis -->
+  <xacro:property name="width" value="0.065" /> <!-- width  is along the x axis -->
+  <xacro:property name="deep" value="0.06" /> <!-- y axis -->
+  <xacro:property name="finger_height" value="0.045" /> <!-- z axis -->
+  <xacro:property name="finger_width" value="0.02" /> <!-- width  is along the x axis -->
+  <xacro:property name="finger_deep" value="0.025" /> <!-- y axis -->
+  <xacro:property name="closing_width" value="0.025" /> <!-- distance between the fingers when closed -->
   <!-- This offset is due to avoid the collision between the gripper and the end effector "boundary"-->
   <xacro:property name="offset" value="0.0051" />

Commit message: minor changes

File: iri_table_clearing_description/xacro/grippertcp.urdf.xacro (robot description, xacro)
@@ -4,10 +4,10 @@
   <xacro:property name="mass" value="0.05" /> <!-- arbitrary value for mass -->
   <xacro:property name="height" value="0.07" /> <!-- z axis -->
-  <xacro:property name="width" value="0.065" /> <!-- width  is along the x axis -->
-  <xacro:property name="deep" value="0.06" /> <!-- y axis -->
+  <xacro:property name="width" value="0.07" /> <!-- width  is along the x axis -->
+  <xacro:property name="deep" value="0.05" /> <!-- y axis -->
   <xacro:property name="finger_height" value="0.045" /> <!-- z axis -->
-  <xacro:property name="finger_width" value="0.02" /> <!-- width  is along the x axis -->
+  <xacro:property name="finger_width" value="0.03" /> <!-- width  is along the x axis -->
   <xacro:property name="finger_deep" value="0.025" /> <!-- y axis -->
-  <xacro:property name="closing_width" value="0.025" /> <!-- distance between the fingers when closed -->
+  <xacro:property name="closing_width" value="0.03" /> <!-- distance between the fingers when closed -->
   <!-- This offset is due to avoid the collision between the gripper and the end effector "boundary"-->
   <xacro:property name="offset" value="0.0051" />
